File: sbc6802.kicad_pcb (KiCad board)
At the start: 2 copper layers, 98.3 x 75.6 mm, 36 parts, among them J1 Conn_02x20_Odd_Even, J2 Conn_01x06, U1 MC6802, U2 74LS04, U3 74LS00, U4 74LS138, U5 28C256 EEPROM, U6 71256 32KB SRAM, U7 PIC12F1822-IP, U8 MC6850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

Commit message: gerber
Parts:
- added G1: LOGO, qr:qr_github_sbc6802, B.Cu at (187.3, 128.3)
Other:
- board text added: "+5V"
- board text added: "0x8"
- board text added: "0xA"
- board text added: "0xE"
- board text added: "A0"
- board text added: "A1"
- board text added: "A14"
- board text added: "A15"
- board text added: "D0"
- board text added: "D1"
- board text added: "D6"
- board text added: "D7"
- board text added: "E"
- board text added: "GND"
- board text added: "NC"
- board text added: "R/~W"
- board text added: "RXD"
- board text added: "TXD"
- board text added: "VMA"
- board text added: "[SBC6802 plus Bus] 2019 RyuStudio"
- board text added: "https://github.com/ryu10/sbc6802"
- board text added: "nc"
- board text added: "~CTS"
- board text added: "~IRQ"
- board text added: "~NMI"
- board text added: "~RD"
- board text added: "~RTS"
- board text added: "~Res"
- board text added: "~WR"
- board text removed: "SBC 6802 plus BUS / 2019 RyuStudio Original Design SBC6800 and SBC6809 / 2017-2018 (c) Tetsuya Suzuki"
- board text removed: "[SBC6802 plus BUS] 2019 RyuStudio"
