File: sbc6802.sch (KiCad schematic (older format))
At the start: 29 parts, among them J1 Conn_02x20_Odd_Even, J2 Conn_01x06, U1 MC6802, U2 74LS04, U3 74LS00, U4 74LS138, U5 28C256 EEPROM, U6 71256 32KB SRAM, U7 PIC12F1822-IP, U8 MC6850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

Commit message: schematics
Other:
- note added: "SBC6802 plus Bus"
- note added: "SBC6802 with SBC Bus Connector \n2019 RyuStudio\n* Derived from SBC6800/SBC6809 (c) 2017-2018 Tetsuya Suzuki\nCC-BY-SA 3.0"
- note removed: "SBC6802 w/Bus"
- note removed: "SBC6802 with SBC Bus Connector \n2019 ryu10\n* Derived from SBC6800/SBC6809 (c) 2017-2018 Tetsuya Suzuki\nCC-BY-SA 3.0"
Changed lines of the file:
@@
 $EndDescr
 Text Notes 7400 7500 0    50   ~ 0
-SBC6802 w/Bus
+SBC6802 plus Bus
 $Comp
 L CPU_NXP_6800:MC6802 U1
@@
 1.0
 Text Notes 7050 7050 0    50   ~ 0
-SBC6802 with SBC Bus Connector \n2019 ryu10\n* Derived from SBC6800/SBC6809 (c) 2017-2018 Tetsuya Suzuki\nCC-BY-SA 3.0
+SBC6802 with SBC Bus Connector \n2019 RyuStudio\n* Derived from SBC6800/SBC6809 (c) 2017-2018 Tetsuya Suzuki\nCC-BY-SA 3.0
 $EndSCHEMATC

Commit message: eesch
Changed lines of the file:
@@
 	1    0    0    -1
 $EndComp
-Wire Wire Line
-	5850 4700 2500 4700
 Connection ~ 6350 3400
 Wire Wire Line
