File: KiCAD/sbc6802.kicad_pcb (KiCad board)
At the start: 2 copper layers, 98.3 x 75.6 mm, 37 parts, among them J1 Conn_02x20_Odd_Even, J2 Conn_01x06, U1 MC6802, U2 74LS04, U3 74LS00, U4 74LS138, U5 28C256 EEPROM, U6 71256 32KB SRAM, U7 PIC12F1822-IP, U8 MC6850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

Commit message: init rev2
Parts:
- removed ? (x3): , 
- removed G1: LOGO, qr:qr_github_sbc6802
- removed MH1, MH2, MH3, MH4: MountingHole_3.2mm_M3, MountingHole:MountingHole_3.2mm_M3
- added mh1: MountingHole_3.2mm_M3, MountingHole:MountingHole_3.2mm_M3, F.Cu at (198.7, 67.2)
- added mh2: MountingHole_3.2mm_M3, MountingHole:MountingHole_3.2mm_M3, F.Cu at (198.7, 132.8)
- added mh3: MountingHole_3.2mm_M3, MountingHole:MountingHole_3.2mm_M3, F.Cu at (109.8, 132.8)
- added mh4: MountingHole_3.2mm_M3, MountingHole:MountingHole_3.2mm_M3, F.Cu at (109.8, 67.2)
- J2: footprint Connector_PinHeader_2.54mm:PinHeader_1x06_P2.54mm_Horizontal -> Connector_PinHeader_2.54mm:PinHeader_1x06_P2.54mm_Vertical; moved to F.Cu
- moved D1 7.85 mm to (131.4, 75.6), turned to 0 degrees
- moved C6 4.45 mm to (117.5, 125.7)
- moved R1 1.91 mm to (131.4, 87.0)
- turned J2 to 270 degrees
Connections:
- J1 pad 32: Net-(J1-Pad32) -> (no net)
- J1 pad 34: Net-(J1-Pad34) -> (no net)
- J1 pad 36: Net-(J1-Pad36) -> (no net)
- J2 pad 4: /P5V -> (no net)
- U1 pad 7: Net-(U1-Pad7) -> (no net)
- U2 pad 11: (no net) -> GND
- U2 pad 13: (no net) -> GND
- U2 pad 9: (no net) -> GND
- U4 pad 12: Net-(U4-Pad12) -> (no net)
- U4 pad 13: Net-(U4-Pad13) -> (no net)
- U4 pad 14: Net-(U4-Pad14) -> (no net)
- U4 pad 15: Net-(U4-Pad15) -> (no net)
- U7 pad 2: Net-(U7-Pad2) -> (no net)
- U7 pad 3: Net-(U7-Pad3) -> (no net)
- U7 pad 4: Net-(U7-Pad4) -> (no net)
- U7 pad 6: Net-(U7-Pad6) -> (no net)
- U7 pad 7: Net-(U7-Pad7) -> (no net)
Routing:
- net GND: track 302.4 -> 0.00 mm
- net +5V: track 251.7 -> 0.00 mm
- net /D0: track 207.2 -> 0.00 mm, vias 1 -> 0
- net /R~W: track 158.8 -> 0.00 mm
- net /~IRQ: track 153.5 -> 0.00 mm, vias 1 -> 0
- net /D5: track 147.1 -> 0.00 mm, vias 2 -> 0
- net /D1: track 144.4 -> 0.00 mm, vias 1 -> 0
- net /A5: track 138.9 -> 0.00 mm
- net /D3: track 134.8 -> 0.00 mm, vias 2 -> 0
- net /A4: track 131.9 -> 0.00 mm
- net /A6: track 128.7 -> 0.00 mm, vias 1 -> 0
- net /E: track 127.9 -> 0.00 mm, vias 2 -> 0
- net /A7: track 127.3 -> 0.00 mm
- net /A8: track 120.3 -> 0.00 mm
- net /D2: track 119.6 -> 0.00 mm, vias 1 -> 0
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- removed copper zone on B.Cu, net GND
- removed copper zone on F.Cu, net GND

Commit message: rev2 pcb & readme
Parts:
- added G***: LOGO, qr:qr_github_sbc6802, B.Cu at (188.0, 128.3)
- moved C11 1.27 mm to (189.9, 107.3)
- moved U7 1.27 mm to (189.9, 111.1)
- moved U8 1.27 mm to (182.2, 75.6)
- moved C12 1.23 mm to (182.3, 107.3)
Routing:
- net GND: track 0.00 -> 331.3 mm
- net +5V: track 0.00 -> 257.4 mm
- net /A0: track 0.00 -> 165.1 mm, vias 0 -> 2
- net /~IRQ: track 0.00 -> 153.2 mm
- net /E: track 0.00 -> 150.0 mm
- net /R~W: track 0.00 -> 149.2 mm
- net /A5: track 0.00 -> 139.1 mm, vias 0 -> 1
- net /D3: track 0.00 -> 135.4 mm
- net /A7: track 0.00 -> 135.1 mm, vias 0 -> 1
- net /A4: track 0.00 -> 130.7 mm
- net /D2: track 0.00 -> 127.3 mm, vias 0 -> 1
- net /A6: track 0.00 -> 121.8 mm, vias 0 -> 1
- net /D1: track 0.00 -> 121.3 mm, vias 0 -> 1
- net /A13: track 0.00 -> 120.4 mm
- net /A3: track 0.00 -> 117.4 mm
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- added copper zone on B.Cu, net GND
- added copper zone on F.Cu, net GND
Other:
- board text added: "[SBC6802 plus Bus] Rev.2 2019 RyuStudio"
- board text removed: "[SBC6802 plus Bus] 2019 RyuStudio"

Commit message: rev2 kicad/gerber
Parts:
- removed G***: LOGO, qr:qr_github_sbc6802
- added logo1: LOGO, qr:qr_github_sbc6802_r2, B.Cu at (187.1, 127.6)
- D1: value DIODE -> D; footprint Diode_THT:D_DO-35_SOD27_P7.62mm_Horizontal -> Diode_THT:D_A-405_P7.62mm_Horizontal
- mh1, mh2, mh3, mh4: value MountingHole_3.2mm_M3 -> M3
- moved C3 1.47 mm to (135.5, 70.9)
- moved C2 1.30 mm to (135.5, 65.9)
- moved mh1 0.52 mm to (198.2, 67.2)
- moved mh2 0.52 mm to (198.2, 132.8)
- moved Y1 0.13 mm to (131.4, 65.9)
Connections:
- D1 pad 1: /~Res -> +5V
- D1 pad 2: +5V -> /~Res
Routing:
- net /A0: track 165.1 -> 104.0 mm, vias 2 -> 0
- net /A6: track 121.8 -> 169.7 mm, vias 1 -> 0
- net /A3: track 117.4 -> 149.9 mm
- net /D6: track 109.8 -> 140.8 mm, vias 1 -> 0
- net /A2: track 92.7 -> 121.6 mm
- net /D7: track 114.6 -> 131.7 mm, vias 0 -> 1
- net /D3: track 135.4 -> 118.9 mm, vias 0 -> 1
- net /~IRQ: track 153.2 -> 136.8 mm, vias 0 -> 1
- net /D0: track 116.6 -> 130.7 mm, vias 1 -> 0
- net /D5: track 111.0 -> 124.2 mm
- net Net-(U3-Pad3): track 67.4 -> 79.1 mm, vias 1 -> 2
- net /A8: track 109.7 -> 121.0 mm
- net /A1: track 93.8 -> 103.4 mm, vias 2 -> 0
- net /D2: track 127.3 -> 120.0 mm, vias 1 -> 0
- net /D4: track 110.1 -> 117.4 mm
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