File: KiCAD/sbc6802.kicad_pcb (KiCad board)
At the start: 2 copper layers, 98.3 x 75.6 mm, 34 parts, among them J1 Conn_02x20_Odd_Even, J2 Conn_01x06, U1 MC6802, U2 74LS04, U3 74LS00, U4 74LS138, U5 28C256 EEPROM, U6 71256 32KB SRAM, U7 PIC12F1822-IP, U8 MC6850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

Commit message: rev2 readme
Other:
- board text added: "A10"
- board text added: "A11"
- board text added: "A12"
- board text added: "A13"
- board text added: "A2"
- board text added: "A3"
- board text added: "A4"
- board text added: "A5"
- board text added: "A6"
- board text added: "A7"
- board text added: "A8"
- board text added: "A9"
- board text added: "D2"
- board text added: "D3"
- board text added: "D4"
- board text added: "D5"
Changed lines of the file:
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@@
   (general
     (thickness 1.6)
-    (drawings 42)
+    (drawings 57)
     (tracks 1305)
     (zones 0)
@@
     (visible_elements FFFFEF7F)
     (pcbplotparams
-      (layerselection 0x010fc_ffffffff)
+      (layerselection 0x010f0_ffffffff)
       (usegerberextensions true)
       (usegerberattributes false)
@@
       (viasonmask false)
       (mode 1)
-      (useauxorigin false)
+      (useauxorigin true)
       (hpglpennumber 1)
       (hpglpenspeed 20)
@@
       (psa4output false)
       (plotreference true)
-      (plotvalue true)
+      (plotvalue false)
       (plotinvisibletext false)
       (padsonsilk false)
@@
     )
   )
-  (target plus (at 104.775 137.795) (size 5) (width 0.05) (layer Edge.Cuts))
+  (gr_text A5 (at 160.147 131.445 90) (layer B.SilkS)
+    (effects (font (size 0.8 0.8) (thickness 0.15)) (justify mirror))
+  )
+  (gr_text A7 (at 157.607 131.445 90) (layer B.SilkS)
+    (effects (font (size 0.8 0.8) (thickness 0.15)) (justify mirror))
+  )
+  (gr_text A3 (at 162.56 131.445 90) (layer B.SilkS)
+    (effects (font (size 0.8 0.8) (thickness 0.15)) (justify mirror))
+  )
+  (gr_text A13 (at 149.86 131.445 90) (layer B.SilkS)
+    (effects (font (size 0.8 0.8) (thickness 0.15)) (justify mirror))
+  )
+  (gr_text A9 (at 154.94 131.318 90) (layer B.SilkS)
+    (effects (font (size 0.8 0.8) (thickness 0.15)) (justify mirror))
+  )
+  (gr_text A11 (at 152.4 131.445 90) (layer B.SilkS)
+    (effects (font (size 0.8 0.8) (thickness 0.15)) (justify mirror))
+  )
+  (gr_text A10 (at 152.4 122.555 90) (layer B.SilkS)
+    (effects (font (size 0.8 0.8) (thickness 0.15)) (justify mirror))
+  )
+  (gr_text A12 (at 149.86 122.555 90) (layer B.SilkS)
+    (effects (font (size 0.8 0.8) (thickness 0.15)) (justify mirror))
+  )
+  (gr_text A8 (at 154.94 122.428 90) (layer B.SilkS)
+    (effects (font (size 0.8 0.8) (thickness 0.15)) (justify mirror))
+  )
+  (gr_text A4 (at 160.147 122.555 90) (layer B.SilkS)
+    (effects (font (size 0.8 0.8) (thickness 0.15)) (justify mirror))
+  )
+  (gr_text A6 (at 157.607 122.555 90) (layer B.SilkS)
+    (effects (font (size 0.8 0.8) (thickness 0.15)) (justify mirror))
+  )
+  (gr_text A2 (at 162.56 122.555 90) (layer B.SilkS)
+    (effects (font (size 0.8 0.8) (thickness 0.15)) (justify mirror))
+  )
+  (gr_text "D3\n" (at 172.72 131.445 90) (layer B.SilkS)
+    (effects (font (size 0.8 0.8) (thickness 0.15)) (justify mirror))
+  )
+  (gr_text D5 (at 170.18 131.445 90) (layer B.SilkS)
+    (effects (font (size 0.8 0.8) (thickness 0.15)) (justify mirror))
+  )
+  (gr_text D4 (at 170.18 122.555 90) (layer B.SilkS)
+    (effects (font (size 0.8 0.8) (thickness 0.15)) (justify mirror))
+  )
+  (gr_text D2 (at 172.72 122.555 90) (layer B.SilkS)
+    (effects (font (size 0.8 0.8) (thickness 0.15)) (justify mirror))
+  )
   (gr_text https://github.com/ryu10/sbc6802 (at 146.05 134.62) (layer B.SilkS)
     (effects (font (size 1.2 1.2) (thickness 0.15)) (justify right mirror))
