File: KiCAD/sbc6802.sch (KiCad schematic (older format))
At the start: 29 parts, among them J1 Conn_02x20_Odd_Even, J2 Conn_01x06, U1 MC6802, U2 74LS04, U3 74LS00, U4 74LS138, U5 28C256 EEPROM, U6 71256 32KB SRAM, U7 PIC12F1822-IP, U8 MC6850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

Commit message: init rev2
Parts:
- added unit 4 of U2
- added unit 5 of U2
- added unit 6 of U2
- J2: footprint Connector_PinHeader_2.54mm:PinHeader_1x06_P2.54mm_Horizontal -> Connector_PinHeader_2.54mm:PinHeader_1x06_P2.54mm_Vertical
Connections:
- net GND: now also U2.11, U2.13, U2.9
- no-connect marks 14 -> 17
Other:
- note added: "2"
- note added: "Dec 1, 2019\n"
- note removed: "1.0"
- note removed: "Nov 14 2019\n"
Changed lines of the file:
@@
 F 0 "J2" H 7980 5792 50  0000 L CNN
 F 1 "Conn_01x06" H 7980 5701 50  0000 L CNN
-F 2 "Connector_PinHeader_2.54mm:PinHeader_1x06_P2.54mm_Horizontal" H 7900 5800 50  0001 C CNN
+F 2 "Connector_PinHeader_2.54mm:PinHeader_1x06_P2.54mm_Vertical" H 7900 5800 50  0001 C CNN
 F 3 "~" H 7900 5800 50  0001 C CNN
 	1    7900 5800
@@
 $EndComp
 Text Notes 8150 7650 0    50   ~ 0
-Nov 14 2019\n
+Dec 1, 2019\n
 Text Notes 10600 7650 0    50   ~ 0
-1.0
+2
 Text Notes 7050 7050 0    50   ~ 0
 SBC6802 with SBC Bus Connector \n2019 RyuStudio\n* Derived from SBC6800/SBC6809 (c) 2017-2018 Tetsuya Suzuki\nCC-BY-SA 3.0
+$Comp
+L 74xx:74LS04 U2
+U 4 1 5DE57A1F
+P 6300 5150
+F 0 "U2" H 6300 5467 50  0000 C CNN
+F 1 "74LS04" H 6300 5376 50  0000 C CNN
+F 2 "Package_DIP:DIP-14_W7.62mm" H 6300 5150 50  0001 C CNN
+F 3 "http://www.ti.com/lit/gpn/sn74LS04" H 6300 5150 50  0001 C CNN
+	4    6300 5150
+	1    0    0    -1
+$EndComp
+$Comp
+L 74xx:74LS04 U2
+U 5 1 5DE5944B
+P 6300 5650
+F 0 "U2" H 6300 5967 50  0000 C CNN
+F 1 "74LS04" H 6300 5876 50  0000 C CNN
+F 2 "Package_DIP:DIP-14_W7.62mm" H 6300 5650 50  0001 C CNN
+F 3 "http://www.ti.com/lit/gpn/sn74LS04" H 6300 5650 50  0001 C CNN
+	5    6300 5650
+	1    0    0    -1
+$EndComp
+$Comp
+L 74xx:74LS04 U2
+U 6 1 5DE5C026
+P 6300 6150
+F 0 "U2" H 6300 6467 50  0000 C CNN
+F 1 "74LS04" H 6300 6376 50  0000 C CNN
+F 2 "Package_DIP:DIP-14_W7.62mm" H 6300 6150 50  0001 C CNN
+F 3 "http://www.ti.com/lit/gpn/sn74LS04" H 6300 6150 50  0001 C CNN
+	6    6300 6150
+	1    0    0    -1
+$EndComp
+Wire Wire Line
+	6000 5150 6000 5650
+Connection ~ 6000 5650
+Wire Wire Line
+	6000 5650 6000 6150
+Connection ~ 6000 6150
+Wire Wire Line
+	6000 6150 6000 6400
+$Comp
+L power:GND #PWR041
+U 1 1 5DE6E439
+P 6000 6400
+F 0 "#PWR041" H 6000 6150 50  0001 C CNN
+F 1 "GND" H 6005 6227 50  0000 C CNN
+F 2 "" H 6000 6400 50  0001 C CNN
+F 3 "" H 6000 6400 50  0001 C CNN
+	1    6000 6400
+	1    0    0    -1
+$EndComp
+NoConn ~ 6600 5150
+NoConn ~ 6600 5650
+NoConn ~ 6600 6150
 $EndSCHEMATC

Commit message: rev2 kicad/gerber
Parts:
- removed D1: DIODE, Diode_THT:D_DO-35_SOD27_P7.62mm_Horizontal, symbol pspice:DIODE
- added D1: D, Diode_THT:D_A-405_P7.62mm_Horizontal, symbol Device:D
Connections:
- net +5V: now also D1.1 (K)
- net ~Res: now also D1.2 (A)
Other:
- note added: "Dec 29, 2019\n"
- note removed: "Dec 1, 2019\n"
Changed lines of the file:
@@
 	1    0    0    -1
 $EndComp
-$Comp
-L pspice:DIODE D1
-U 1 1 5E73D19A
-P 800 3400
-F 0 "D1" V 1200 3500 50  0000 R CNN
-F 1 "DIODE" V 1100 3500 50  0000 R CNN
-F 2 "Diode_THT:D_DO-35_SOD27_P7.62mm_Horizontal" H 800 3400 50  0001 C CNN
-F 3 "~" H 800 3400 50  0001 C CNN
-	1    800  3400
-	0    -1   -1   0
-$EndComp
-Wire Wire Line
-	1050 3100 1050 3200
-Wire Wire Line
-	800  3200 1050 3200
 Wire Wire Line
 	800  3600 1050 3600
-Connection ~ 1050 3200
-Wire Wire Line
-	1050 3200 1050 3300
 $Comp
 L Device:R R1
@@
 $EndComp
 Text Notes 8150 7650 0    50   ~ 0
-Dec 1, 2019\n
+Dec 29, 2019\n
 Text Notes 10600 7650 0    50   ~ 0
 2
@@
 NoConn ~ 6600 5650
 NoConn ~ 6600 6150
+$Comp
+L Device:D D1
+U 1 1 5E0A982D
+P 800 3450
+F 0 "D1" V 754 3529 50  0000 L CNN
+F 1 "D" V 845 3529 50  0000 L CNN
+F 2 "Diode_THT:D_A-405_P7.62mm_Horizontal" H 800 3450 50  0001 C CNN
+F 3 "~" H 800 3450 50  0001 C CNN
+	1    800  3450
+	0    1    1    0
+$EndComp
+Wire Wire Line
+	1050 3100 1050 3300
+Wire Wire Line
+	1050 3300 800  3300
+Connection ~ 1050 3300
 $EndSCHEMATC
